File: pcb/pcb.sch (KiCad schematic (older format))
At the start: 18 parts, among them J1 processor_right, J2 processor_left, J3 GSM, J4 charger, J5 sensors, J6 BME_280, J7 debug_pwr_jumper

Commit message: Fixes.
Parts:
- R9: value 20k -> 22k
Other:
- note removed: "TODO: RST"
Changed lines of the file:
@@
 P 2600 5600
 F 0 "R9" V 2796 5600 50  0000 C CNN
-F 1 "20k" V 2705 5600 50  0000 C CNN
+F 1 "22k" V 2705 5600 50  0000 C CNN
 F 2 "Resistor_THT:R_Axial_DIN0207_L6.3mm_D2.5mm_P10.16mm_Horizontal" H 2600 5600 50  0001 C CNN
 F 3 "~" H 2600 5600 50  0001 C CNN
@@
 Text GLabel 8550 1000 0    50   Input ~ 0
 PROC_RESET
-Text Notes 4500 1700 0    50   ~ 0
-TODO: RST
 Text Label 6250 1950 2    50   ~ 0
 RX
